File: TCD1304Rev2KiCAD/TCD1304Rev2.kicad_pcb (KiCad board)
At the start: 4 copper layers, 60 x 40 mm, 26 parts, among them J1 Conn_01x08_Male, J2 Conn_01x16_Male, U1 TCD1304AP, U2 ADA4807-2, U3 Teensy4.0

Commit message: Correction
C7 should be 68p and DNP (do not populate).    Normally, for a SAR type input,  best results are obtain with an external resistor and capacitor to act as a charge reservoir for the sampling capacitor.    But, the analog inputs of microcontrollers used in Teensy, Arduino, SMT, etc., typically have a large resistance in series with the sampling capacitor.  This large resistance preempts any benefit from the external capacitor and instead lengthens the time constant for charging the sampling capacitor.   In this revision, we replace the external cap with one having a smaller value and we mark it as do-not-populate.   Indeed it should be left not populated.
Parts:
- C7: value 1nF -> 68p
- R3: value 2.5K -> 2.49K
- U2: value ADA4807-2 -> ADA4807-2ARMZ-R7

Commit message: Minor changes (best practice update)
Parts:
- moved J1 0.50 mm to (173.2, 117.5)
- moved J2 0.50 mm to (177.1, 82.5)
- moved C4 0.06 mm to (130.7, 103.5)
Routing:
- net Earth: track 17.2 -> 16.3 mm, vias 7 -> 8
- net +3.3V: track 15.4 -> 14.7 mm
- net Net-(J2-Pin_6): track 41.7 -> 41.0 mm
- net Net-(J2-Pin_5): track 10.6 -> 9.92 mm
- net Net-(J2-Pin_8): track 25.2 -> 24.7 mm
- net Net-(J2-Pin_4): track 10.6 -> 10.1 mm
- net Net-(J2-Pin_3): track 10.6 -> 10.1 mm
- net Net-(J2-Pin_2): track 10.6 -> 10.1 mm
- net Net-(J2-Pin_15): track 27.2 -> 26.7 mm
- net Net-(J2-Pin_12): track 10.6 -> 10.1 mm
- net Net-(J1-Pin_7): track 4.99 -> 4.49 mm
- net Net-(J1-Pin_5): track 4.78 -> 4.28 mm
Other:
- board text added: "TCD1304 Rev2b Mitchell C Nelson, PhD Dec 26, 2024"
- board text removed: "D0"
- board text removed: "D13"
- board text removed: "D3"
- board text removed: "D8"
- board text removed: "ICG"
- board text removed: "SH"
- board text removed: "TCD1304 Rev2 Mitchell C Nelson, PhD Jan 30, 2023"
- board text removed: "fMClk"
