File: TCD1304Rev2KiCAD/TCD1304Rev2.kicad_sch (KiCad schematic)
At the start: 26 parts, among them J1 Conn_01x08_Male, J2 Conn_01x16_Male, U1 TCD1304AP, U2 ADA4807-2ARMZ-R7, U3 Teensy4.0

Commit message: Minor changes (best practice update)
Parts:
- C7: value 1nF -> 68p; Digikey 399-17840-1-ND -> 1276-1135-1-ND; now not fitted
Other:
- moved on the sheet: C3, C4
